File: Board V4/DecodingBoard/DecodingBoard.kicad_pcb (KiCad board)
At the start: 4 copper layers, 47.5 x 41 mm, 71 parts, among them IC1 STM32WBA65CIU6, IC2 RN4871-V_RM140, IC3 MCP111-195I_TO, J1 UJ20-C-H-G-SMT-1-P16-TR, J3 TSM-106-02-T-SH-LC, J4 2053380004, J5 5037630691, J6 5040500691, SW1 TL3305BF100QG, SW2 TL3305BF100QG, U1 ESDS302DBVR, U2 TPS7A7200RGWT, U3 USBLC6-2SC6, U4 TPS2121RUXR

Commit message: Changed J5 part number
Parts:
- J4: value 2053380004 -> 2053380002
- J5: value 5037630691 -> 5037630491
Changed lines of the file:
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@@
 			)
 		)
-		(property "Value" "5037630691"
+		(property "Value" "5037630491"
 			(at 0 2.4343 0)
 			(unlocked yes)
@@
 			)
 		)
-		(property "Datasheet" "https://www.molex.com/en-us/products/part-detail-pdf/5037630691?display=pdf"
+		(property "Datasheet" "https://www.molex.com/en-us/products/part-detail/5037630491"
 			(at 0 0 0)
 			(layer "F.Fab")
@@
 			)
 		)
-		(property "Value" "2053380004"
+		(property "Value" "2053380002"
 			(at 0 3.727702 90)
 			(unlocked yes)
@@
 			)
 		)
-		(property "Datasheet" "https://www.molex.com/en-us/products/part-detail-pdf/2053380004?display=pdf"
+		(property "Datasheet" "https://www.molex.com/en-us/products/part-detail-pdf/2053380002?display=pdf"
 			(at 0 0 90)
 			(layer "F.Fab")
@@
 		(net "GND")
 		(layer "B.Cu")
-		(hatch full 0.5)
+		(hatch edge 0.5)
 		(priority 2)
 		(connect_pads

Commit message: Added keep-out zone under ble module as per datasheet recommendation
Routing:
- net Net-(IC2-RST_N): track 17.0 -> 20.2 mm
- net Net-(IC2-P2_0): track 5.04 -> 5.72 mm
Changed lines of the file:
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@@
 	)
 	(segment
+		(start 101.1 54)
+		(end 101.1 55.0343)
+		(width 0.5)
+		(layer "F.Cu")
+		(net "+5V")
+	)
+	(segment
 		(start 122.5 69)
 		(end 122.8 68.7)
@@
 	)
 	(segment
-		(start 101.1 54)
-		(end 101.1 55.0343)
-		(width 0.5)
-		(layer "F.Cu")
-		(net "+5V")
-	)
-	(segment
 		(start 121.95 67)
 		(end 121.462411 67)
@@
 	)
 	(segment
-		(start 108 81)
-		(end 109.85 81)
+		(start 111.32 80.85)
+		(end 111.33 80.86)
+		(width 0.3)
+		(layer "F.Cu")
+		(net "Net-(IC2-RST_N)")
+	)
+	(segment
+		(start 110 80.85)
+		(end 111.32 80.85)
 		(width 0.3)
 		(layer "F.Cu")
@@
 	)
 	(via
-		(at 108 81)
+		(at 111.33 80.86)
 		(size 0.6)
 		(drill 0.3)
@@
 	)
 	(segment
+		(start 107.73 72.89)
+		(end 111.33 76.49)
+		(width 0.3)
+		(layer "B.Cu")
+		(net "Net-(IC2-RST_N)")
+	)
+	(segment
 		(start 100.82 70.26)
 		(end 102.08 71.52)
@@
 	(segment
 		(start 102.08 71.52)
-		(end 102.08 75.08)
+		(end 103.45 72.89)
 		(width 0.3)
 		(layer "B.Cu")
@@
 	)
 	(segment
-		(start 102.08 75.08)
-		(end 108 81)
+		(start 103.45 72.89)
+		(end 107.73 72.89)
 		(width 0.3)
 		(layer "B.Cu")
@@
 	)
 	(segment
+		(start 111.33 76.49)
+		(end 111.33 80.86)
+		(width 0.3)
+		(layer "B.Cu")
+		(net "Net-(IC2-RST_N)")
+	)
+	(segment
 		(start 109.5 77.5)
 		(end 109.3 77.5)
@@
 	)
 	(segment
-		(start 103.6 78.4)
-		(end 102.8 78.4)
-		(width 0.3)
+		(start 103.6 77.248578)
+		(end 103.6 78.4)
+		(width 0.2)
 		(layer "F.Cu")
 		(net "Net-(IC2-P2_0)")
 	)
 	(segment
-		(start 102.8 78.4)
-		(end 99.8 75.4)
-		(width 0.3)
+		(start 99.8 75.4)
+		(end 101.751422 75.4)
+		(width 0.2)
+		(layer "F.Cu")
+		(net "Net-(IC2-P2_0)")
+	)
+	(segment
+		(start 101.751422 75.4)
+		(end 103.6 77.248578)
+		(width 0.2)
 		(layer "F.Cu")
 		(net "Net-(IC2-P2_0)")
@@
 	)
 	(zone
+		(layers "F.Cu" "B.Cu" "In1.Cu" "In2.Cu")
+		(name "BLE_KEEPOUT_1")
+		(hatch edge 0.5)
+		(connect_pads
+			(clearance 0)
+		)
+		(min_thickness 0.15)
+		(keepout
+			(tracks not_allowed)
+			(vias not_allowed)
+			(pads not_allowed)
+			(copperpour not_allowed)
+			(footprints allowed)
+		)
+		(placement
+			(enabled no)
+			(sheetname "/")
+		)
+		(fill
+			(thermal_gap 0.4)
+			(thermal_bridge_width 0.25)
+			(smoothing fillet)
+			(radius 0.5)
+			(island_removal_mode 0)
+		)
+		(polygon
+			(pts
+				(xy 102.87 79.42) (xy 108.88 79.42) (xy 108.9 85.93) (xy 102.87 85.91) (xy 102.89 85.87)
+			)
+		)
+	)
+	(zone
+		(layers "F.Cu" "B.Cu" "In1.Cu" "In2.Cu" "Edge.Cuts")
+		(name "BLE_KEEPOUT")
+		(hatch edge 0.5)
+		(connect_pads
+			(clearance 0)
+		)
+		(min_thickness 0.15)
+		(keepout
+			(tracks not_allowed)
+			(vias not_allowed)
+			(pads not_allowed)
+			(copperpour not_allowed)
+			(footprints allowed)
+		)
+		(placement
+			(enabled no)
+			(sheetname "/")
+		)
+		(fill
+			(thermal_gap 0.4)
+			(thermal_bridge_width 0.25)
+			(smoothing fillet)
+			(radius 0.5)
+			(island_removal_mode 0)
+		)
+		(polygon
+			(pts
+				(xy 102.87 76.66) (xy 97.5 76.65) (xy 97.51 89.5) (xy 102.9 89.49)
+			)
+		)
+	)
+	(zone
 		(net "GND")
 		(layer "B.Cu")
@@
 			(smoothing fillet)
 			(radius 0.5)
-			(island_removal_mode 1)
+			(island_removal_mode 0)
 		)
 		(polygon
