File: Board V4/DecodingBoard/I2C.kicad_sch (KiCad schematic)
At the start: 3 parts, among them J5 5037630691

Commit message: Changed J5 part number
Parts:
- J5: value 5037630691 -> 5037630491
Changed lines of the file:
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@@
 			)
 		)
-		(property "Value" "5037630691"
+		(property "Value" "5037630491"
 			(at 29.21 29.21 0)
 			(show_name no)
@@
 			)
 		)
-		(property "Datasheet" "https://www.molex.com/en-us/products/part-detail-pdf/5037630691?display=pdf"
+		(property "Datasheet" "https://www.molex.com/en-us/products/part-detail/5037630491"
 			(at 38.1 46.99 0)
 			(hide yes)
