File: Board V4/DecodingBoard/DecodingBoard.kicad_sch (KiCad schematic)
At the start: 22 parts, among them IC1 STM32WBA65CIU6, J3 TSM-106-02-T-SH-LC, J4 2053380004, J6 5040500691, SW1 TL3305BF100QG, SW2 TL3305BF100QG, U1 ESDS302DBVR

Commit message: Changed J4 to correct part number
Parts:
- J4: value 2053380004 -> 2053380002
Changed lines of the file:
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@@
 			)
 		)
-		(property "Value" "2053380004"
+		(property "Value" "2053380002"
 			(at 55.626 169.164 0)
 			(show_name no)
@@
 			)
 		)
-		(property "Datasheet" "https://www.molex.com/en-us/products/part-detail-pdf/2053380004?display=pdf"
+		(property "Datasheet" "https://www.molex.com/en-us/products/part-detail-pdf/2053380002?display=pdf"
 			(at 55.88 182.88 0)
 			(hide yes)

Commit message: Changed USB-C symbol to match new connector
Parts:
- H1, H2: Added to order (none) -> NA; Customer PN (none) -> NA

Commit message: [fix]: reviewed decoding board. Modified J6 connector to 3 pin 1mm pitch Picko-Lock and routed the differential USB
Parts:
- J6: value 5040500691 -> 5037630391; footprint Footprints:CONN_5040500491_MOL -> Footprints:5037630391
Connections:
- net GND: no longer J6.6
Changed lines of the file:
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@@
-	)
-	(junction
-		(at 41.91 74.93)
-		(diameter 0)
-		(color 0 0 0 0)
 	)
 	(junction
@@
 	(wire
 		(pts
-			(xy 41.91 72.39) (xy 41.91 74.93)
-		)
-		(stroke
-			(width 0)
-			(type default)
-		)
-	)
-	(wire
-		(pts
 			(xy 165.1 144.78) (xy 165.1 156.21)
 		)
@@
 		(pts
 			(xy 266.7 74.93) (xy 207.01 74.93)
-		)
-		(stroke
-			(width 0)
-			(type default)
-		)
-	)
-	(wire
-		(pts
-			(xy 39.37 72.39) (xy 41.91 72.39)
 		)
 		(stroke
@@
 			)
 		)
-		(property "Value" "5040500691"
+		(property "Value" "5037630391"
 			(at 30.48 67.31 0)
 			(show_name no)
@@
 			)
 		)
-		(property "Footprint" "Footprints:CONN_5040500491_MOL"
+		(property "Footprint" "Footprints:5037630391"
 			(at 39.37 85.09 0)
 			(hide yes)
@@
 		)
 		(property "Datasheet" "https://www.molex.com/en-us/products/part-detail-pdf/5040500691?display=pdf"
-			(at 39.37 85.09 0)
+			(at 37.084 90.424 0)
 			(hide yes)
 			(show_name no)
@@
 		(pin "5"
 		)
-		(pin "6"
-		)
 		(pin "4"
