File: POWERBOARD v3/power_v3.3/Conversion battery-5.3V_v3.3.kicad_sch (KiCad schematic)
At the start: 11 parts, among them U3 TPS62160DSG

Commit message: Made BOM with Customer PNs
Parts:
- BUCK5V3, GND1, SYS1: Added to order (none) -> NA; Customer PN (none) -> NA
- Cin1: Added to order (none) -> Y; Customer PN (none) -> EMG-PWR-037
- Cout1: Added to order (none) -> Y; Customer PN (none) -> EMG-PWR-040A
- L2: Added to order (none) -> Y; Customer PN (none) -> EMG-PWR-032
- R10: Added to order (none) -> Y; Customer PN (none) -> EMG-PWR-039
- R11: Added to order (none) -> Y; Customer PN (none) -> EMG-PWR-024
- R12: Added to order (none) -> Y; Customer PN (none) -> EMG-PWR-023
- S1: Added to order (none) -> Y; Customer PN (none) -> EMG-PWR-013
- U3: Added to order (none) -> Y; Customer PN (none) -> EMG-PWR-017

Commit message: Added test point footprints
Parts:
- BUCK5V3, GND1, SYS1: Added to order NA -> (none); Customer PN NA -> EMG-PWR-042
Changed lines of the file:
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@@
 			)
 		)
-		(property "Added to order" "NA"
+		(property "Added to order" ""
 			(at 152.4 125.73 0)
 			(hide yes)
@@
 			)
 		)
-		(property "Customer PN" "NA"
+		(property "Customer PN" "EMG-PWR-042"
 			(at 152.4 125.73 0)
 			(hide yes)
@@
 			)
 		)
-		(property "Added to order" "NA"
+		(property "Added to order" ""
 			(at 54.61 90.17 0)
 			(hide yes)
@@
 			)
 		)
-		(property "Customer PN" "NA"
+		(property "Customer PN" "EMG-PWR-042"
 			(at 54.61 90.17 0)
 			(hide yes)
@@
 			)
 		)
-		(property "Added to order" "NA"
+		(property "Added to order" ""
 			(at 204.47 74.93 0)
 			(hide yes)
@@
 			)
 		)
-		(property "Customer PN" "NA"
+		(property "Customer PN" "EMG-PWR-042"
 			(at 204.47 74.93 0)
 			(hide yes)
