File: BioAmp_V2/BioAmp-EXG-Pill.kicad_sch (KiCad schematic)
At the start: 41 parts, among them IC1 ADS112C04IPW, J1 Conn_01x06_Pin, J2 Conn_01x06_Pin, J4 522710469, U1 TL074HIPWR

Commit message: Changed DRL resistors to 1M + 1.5M in series, added .history to gitignore.
Parts:
- R11: value 1M -> 1.5M; Distributer Link https://www.mouser.ch/en/ProductDetail/Bourns/CRT0603-BZ-10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 -> (none)
- R15: value 22K -> 1M; Distributer Link https://www.mouser.ch/en/ProductDetail/YAGEO/RC0603FR-1022K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 -> (none)
Changed lines of the file:
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@@
 			)
 		)
-		(property "Value" "1M"
+		(property "Value" "1.5M"
 			(at 119.38 161.29 90)
 			(show_name no)
@@
 			)
 		)
-		(property "Distributer Link" "https://www.mouser.ch/en/ProductDetail/Bourns/CRT0603-BZ-1004ELF?qs=pxDZlBjcsCiRaiGe6sfQhA%3D%3D"
+		(property "Distributer Link" ""
 			(at 119.38 161.29 90)
 			(hide yes)
@@
 			)
 		)
-		(property "Value" "22K"
+		(property "Value" "1M"
 			(at 109.22 161.29 90)
 			(show_name no)
@@
 			)
 		)
-		(property "Distributer Link" "https://www.mouser.ch/en/ProductDetail/YAGEO/RC0603FR-1022KL?qs=EiqXWrxQq61e6RoATMUfKw%3D%3D"
+		(property "Distributer Link" ""
 			(at 109.22 161.29 90)
 			(hide yes)

Commit message: changed DRL resistors to 1M and 1.8M in series for stricter current limiting.
Parts:
- R11: value 1.5M -> 1.8M
Changed lines of the file:
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@@
 			)
 		)
-		(property "Value" "1.5M"
+		(property "Value" "1.8M"
 			(at 119.38 161.29 90)
 			(show_name no)
